File: arduino_uno.kicad_pcb (KiCad board)
At the start: 2 copper layers, 43 x 32 mm, 18 parts, among them J1 Conn_01x06, J2 Conn_01x12, J4 Conn_01x12, SW1 SW_Push, U1 MIC5205-5.0YM5, U2 ATmega328P-A, Y1 Resonator_Small

Commit message: second commit
Routing:
- net VCC: track 84.3 -> 80.5 mm
Changed lines of the file:
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@@
   (segment (start 140.94 70.825) (end 140.825 70.825) (width 0.25) (layer "F.Cu") (net 1))
   (segment (start 141.065 70.95) (end 140.94 70.825) (width 0.25) (layer "F.Cu") (net 1))
-  (segment (start 140.825 70.825) (end 139.115 69.115) (width 0.25) (layer "F.Cu") (net 1))
+  (segment (start 140.824991 70.825004) (end 139.115013 69.115) (width 0.6096) (layer "F.Cu") (net 1))
   (segment (start 143.025 68.8875) (end 142.8625 69.05) (width 0.25) (layer "F.Cu") (net 1))
-  (segment (start 139.115 67.885) (end 141 66) (width 0.25) (layer "F.Cu") (net 1))
-  (segment (start 143.025 66) (end 143.025 68.8875) (width 0.25) (layer "F.Cu") (net 1))
-  (segment (start 142.8625 70.95) (end 141.065 70.95) (width 0.25) (layer "F.Cu") (net 1))
-  (segment (start 141 66) (end 143.025 66) (width 0.25) (layer "F.Cu") (net 1))
-  (segment (start 139.115 69.115) (end 139.115 67.885) (width 0.25) (layer "F.Cu") (net 1))
+  (segment (start 139.115013 67.885005) (end 140.999997 65.999995) (width 0.6096) (layer "F.Cu") (net 1))
+  (segment (start 143.025012 65.999995) (end 143.025012 68.887492) (width 0.6096) (layer "F.Cu") (net 1))
+  (segment (start 142.862503 70.949998) (end 141.064996 70.949998) (width 0.6096) (layer "F.Cu") (net 1))
+  (segment (start 140.999997 65.999995) (end 143.025012 65.999995) (width 0.6096) (layer "F.Cu") (net 1))
+  (segment (start 139.115013 69.115) (end 139.115013 67.885005) (width 0.6096) (layer "F.Cu") (net 1))
   (segment (start 157.958406 79.45272) (end 157.529605 79.45272) (width 0.25) (layer "F.Cu") (net 2))
   (segment (start 157.716676 81.473732) (end 160.790952 84.548008) (width 0.25) (layer "F.Cu") (net 2))
   (segment (start 157 80.757056) (end 157.716676 81.473732) (width 0.25) (layer "F.Cu") (net 2))
-  (segment (start 166 77.7875) (end 163.4475 80.34) (width 0.25) (layer "F.Cu") (net 2))
-  (segment (start 169.225 76) (end 169.225 77) (width 0.25) (layer "F.Cu") (net 2))
   (segment (start 157 79.982325) (end 157 80.757056) (width 0.25) (layer "F.Cu") (net 2))
-  (segment (start 169.225 76) (end 169.225 73) (width 0.25) (layer "F.Cu") (net 2))
-  (segment (start 141.665 70) (end 142.8625 70) (width 0.25) (layer "F.Cu") (net 2))
+  (segment (start 168.437509 77.7875) (end 165.6825 77.7875) (width 0.6096) (layer "F.Cu") (net 2))
+  (segment (start 169.225011 76.999998) (end 168.437509 77.7875) (width 0.6096) (layer "F.Cu") (net 2))
+  (segment (start 141.664995 70.000012) (end 142.862503 70.000012) (width 0.6096) (layer "F.Cu") (net 2))
   (segment (start 151.184314 73.81) (end 152.271953 74.897639) (width 0.25) (layer "F.Cu") (net 2))
-  (segment (start 168.4375 77.7875) (end 166 77.7875) (width 0.25) (layer "F.Cu") (net 2))
-  (segment (start 140.94 69.275) (end 141.665 70) (width 0.25) (layer "F.Cu") (net 2))
+  (segment (start 140.940003 69.274995) (end 141.664995 70.000012) (width 0.6096) (layer "F.Cu") (net 2))
   (segment (start 158.848047 80.342361) (end 157.958406 79.45272) (width 0.25) (layer "F.Cu") (net 2))
+  (segment (start 169.225011 73.000006) (end 169.225011 76.999998) (width 0.6096) (layer "F.Cu") (net 2))
   (segment (start 150.24 73.81) (end 151.184314 73.81) (width 0.25) (layer "F.Cu") (net 2))
+  (segment (start 165.6825 77.7875) (end 163.13 80.34) (width 0.6096) (layer "F.Cu") (net 2))
   (segment (start 160.790952 84.548008) (end 162.548008 84.548008) (width 0.25) (layer "F.Cu") (net 2))
-  (segment (start 163.4475 80.34) (end 163.13 80.34) (width 0.25) (layer "F.Cu") (net 2))
   (segment (start 162.548008 84.548008) (end 163.096016 84) (width 0.25) (layer "F.Cu") (net 2))
   (segment (start 157.529605 79.45272) (end 157 79.982325) (width 0.25) (layer "F.Cu") (net 2))
-  (segment (start 169.225 77) (end 168.4375 77.7875) (width 0.25) (layer "F.Cu") (net 2))
   (segment (start 163.096016 84) (end 167 84) (width 0.25) (layer "F.Cu") (net 2))
   (via (at 167 84) (size 0.8) (drill 0.4) (layers "F.Cu" "B.Cu") (net 2))
   (segment (start 167 84) (end 167 78.65) (width 0.25) (layer "B.Cu") (net 2))
   (segment (start 167 78.65) (end 174 71.65) (width 0.25) (layer "B.Cu") (net 2))
-  (segment (start 160 82) (end 160.818528 81.181472) (width 0.25) (layer "F.Cu") (net 3))
-  (segment (start 162.637056 83) (end 167.73 83) (width 0.25) (layer "F.Cu") (net 3))
-  (segment (start 149.818427 69.05) (end 146.05 69.05) (width 0.25) (layer "F.Cu") (net 3))
+  (segment (start 160.00001 81.999988) (end 160.818525 81.181473) (width 0.6096) (layer "F.Cu") (net 3))
+  (segment (start 162.637064 83.000012) (end 167.729992 83.000012) (width 0.6096) (layer "F.Cu") (net 3))
   (segment (start 140.65 74.955) (end 140.65 73.3575) (width 0.25) (layer "F.Cu") (net 3))
-  (segment (start 150.645 66) (end 150.645 68.1775) (width 0.25) (layer "F.Cu") (net 3))
-  (segment (start 174 76.73) (end 171.505 76.73) (width 0.25) (layer "F.Cu") (net 3))
-  (segment (start 170.775 73) (end 170.775 76) (width 0.25) (layer "F.Cu") (net 3))
-  (segment (start 149.7725 69.05) (end 146.05 69.05) (width 0.25) (layer "F.Cu") (net 3))
-  (segment (start 159.374314 82) (end 158.282361 80.908047) (width 0.25) (layer "F.Cu") (net 3))
-  (segment (start 153.96901 73.200583) (end 149.818427 69.05) (width 0.25) (layer "F.Cu") (net 3))
-  (segment (start 160 82) (end 161.451992 83.451992) (width 0.25) (layer "F.Cu") (net 3))
+  (segment (start 160 82) (end 159.374319 82) (width 0.6096) (layer "F.Cu") (net 3))
+  (segment (start 174.000008 76.729996) (end 171.504991 76.729996) (width 0.6096) (layer "F.Cu") (net 3))
+  (segment (start 150.645012 68.177512) (end 149.772497 69.050002) (width 0.6096) (layer "F.Cu") (net 3))
+  (segment (start 170.774995 73.000006) (end 170.774995 76) (width 0.6096) (layer "F.Cu") (net 3))
+  (segment (start 153.969009 73.20059) (end 149.81842 69.050002) (width 0.6096) (layer "F.Cu") (net 3))
+  (segment (start 160.00001 81.999988) (end 161.452001 83.451979) (width 0.6096) (layer "F.Cu") (net 3))
   (segment (start 143.67 75.175) (end 145.295 75.175) (width 0.25) (layer "F.Cu") (net 3))
-  (segment (start 171.505 76.73) (end 170.775 76) (width 0.25) (layer "F.Cu") (net 3))
-  (segment (start 153.96901 73.200583) (end 154.200583 73.200583) (width 0.25) (layer "F.Cu") (net 3))
-  (segment (start 146.05 69.05) (end 145.1375 69.05) (width 0.25) (layer "F.Cu") (net 3))
-  (segment (start 154.200583 73.200583) (end 156 75) (width 0.25) (layer "F.Cu") (net 3))
+  (segment (start 171.504991 76.729996) (end 170.774995 76) (width 0.6096) (layer "F.Cu") (net 3))
+  (segment (start 155.768429 75.000002) (end 155.999993 75.000002) (width 0.6096) (layer "F.Cu") (net 3))
+  (segment (start 153.96901 73.200583) (end 155.768429 75.000002) (width 0.6096) (layer "F.Cu") (net 3))
+  (segment (start 145.137502 69.050002) (end 145.1375 69.05) (width 0.6096) (layer "F.Cu") (net 3))
   (segment (start 140.65 73.3575) (end 140.3925 73.1) (width 0.25) (layer "F.Cu") (net 3))
   (segment (start 140.65 74.955) (end 143.45 74.955) (width 0.25) (layer "F.Cu") (net 3))
-  (segment (start 159.413732 79.776676) (end 160.818528 81.181472) (width 0.25) (layer "F.Cu") (net 3))
+  (segment (start 159.413727 79.776676) (end 160.818525 81.181473) (width 0.6096) (layer "F.Cu") (net 3))
+  (segment (start 150.645012 65.999995) (end 150.645012 68.177512) (width 0.6096) (layer "F.Cu") (net 3))
   (segment (start 145.275 80.615) (end 145.61 80.95) (width 0.25) (layer "F.Cu") (net 3))
   (segment (start 145.275 75.025) (end 145.275 80.615) (width 0.25) (layer "F.Cu") (net 3))
   (segment (start 143.45 74.955) (end 143.67 75.175) (width 0.25) (layer "F.Cu") (net 3))
   (segment (start 145.295 75.175) (end 145.36 75.11) (width 0.25) (layer "F.Cu") (net 3))
-  (segment (start 167.73 83) (end 174 76.73) (width 0.25) (layer "F.Cu") (net 3))
-  (segment (start 150.645 68.1775) (end 149.7725 69.05) (width 0.25) (layer "F.Cu") (net 3))
-  (segment (start 160 82) (end 159.374314 82) (width 0.25) (layer "F.Cu") (net 3))
-  (segment (start 160.818528 81.181472) (end 162.637056 83) (width 0.25) (layer "F.Cu") (net 3))
+  (segment (start 167.729992 83.000012) (end 174.000008 76.729996) (width 0.6096) (layer "F.Cu") (net 3))
+  (segment (start 149.772497 69.050002) (end 145.137502 69.050002) (width 0.6096) (layer "F.Cu") (net 3))
+  (segment (start 159.374319 82) (end 158.282361 80.908042) (width 0.6096) (layer "F.Cu") (net 3))
+  (segment (start 160.818525 81.181473) (end 162.637064 83.000012) (width 0.6096) (layer "F.Cu") (net 3))
   (via (at 145.275 75.025) (size 0.8) (drill 0.4) (layers "F.Cu" "B.Cu") (net 3))
   (via (at 156 75) (size 0.8) (drill 0.4) (layers "F.Cu" "B.Cu") (net 3))
@@
   (segment (start 145.275 71.285) (end 145.275 75.025) (width 0.25) (layer "B.Cu") (net 3))
   (segment (start 150.645 66) (end 150.56 66) (width 0.25) (layer "B.Cu") (net 3))
-  (segment (start 157 75) (end 160 78) (width 0.25) (layer "B.Cu") (net 3))
-  (segment (start 160 78) (end 160 82) (width 0.25) (layer "B.Cu") (net 3))
-  (segment (start 156 75) (end 157 75) (width 0.25) (layer "B.Cu") (net 3))
+  (segment (start 156.999991 75.000002) (end 160.00001 77.999996) (width 0.6096) (layer "B.Cu") (net 3))
+  (segment (start 160.00001 77.999996) (end 160.00001 81.999988) (width 0.6096) (layer "B.Cu") (net 3))
+  (segment (start 155.999993 75.000002) (end 156.999991 75.000002) (width 0.6096) (layer "B.Cu") (net 3))
   (segment (start 150.56 66) (end 145.275 71.285) (width 0.25) (layer "B.Cu") (net 3))
   (segment (start 152.837639 74.331953) (end 152.837639 74.215607) (width 0.25) (layer "F.Cu") (net 4))
